File: 68v2.kicad_pcb (KiCad board)
At the start: 2 copper layers, 328.7 x 101.6 mm, 138 parts, among them J1 Columns, J2 Rows

Commit message: Better columns
Parts:
- moved J1 25.5 mm to (169.9, 14.3)
- moved J2 12.7 mm to (177.8, 14.3)
Routing:
- net ROW4: track 231.6 -> 99.5 mm, vias 1 -> 0
- net COL1: track 577.9 -> 456.9 mm
- net ROW5: track 236.4 -> 119.9 mm, vias 1 -> 0
- net ROW6: track 201.4 -> 108.6 mm, vias 1 -> 0
- net COL2: track 510.1 -> 422.1 mm
- net ROW3: track 224.4 -> 139.6 mm, vias 1 -> 0
- net ROW2: track 207.1 -> 133.3 mm, vias 1 -> 0
- net ROW7: track 140.7 -> 69.0 mm, vias 1 -> 0
- net COL3: track 337.8 -> 277.7 mm
- net ROW8: track 194.6 -> 140.5 mm, vias 1 -> 0
- net ROW1: track 174.7 -> 130.9 mm, vias 1 -> 0
- net COL4: track 349.3 -> 307.6 mm
- net ROW9: track 185.8 -> 152.3 mm, vias 1 -> 0
- net ROW0: track 154.5 -> 126.2 mm, vias 1 -> 0
- net COL5: track 310.5 -> 286.9 mm
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Other:
- board size 328.7 x 101.6 mm -> 328.7 x 100.6 mm
