File: dev-68.sch (KiCad schematic (older format))
At the start: 212 parts, among them J1 POWER, J2 ROWS, J3 COLUMNS, J4 LED DRIVERS, U1 IS31FL3733-QF, U2 IS31FL3733-QF

Commit message: Rename project to dev-68.
Parts:
- D101, D102, D103, D104, D105, D106, D107, D108, D109, D110, D111, D112, D113, D114, D115, D116, D117, D118, D119, D120, D121, D122, D123, D124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: footprint xebow:Wurth_PLCC6 -> dev-68:Wurth_PLCC6; symbol Device:LED_RGB -> dev-68:LED_RGB_BRG
