File: dev-68.sch (KiCad schematic (older format))
At the start: 208 parts, among them J1 Columns, J2 Rows, U1 IS31FL3733-TQ, U2 IS31FL3733-TQ

Commit message: Some tracing
Parts:
- added J3: RGB LED Matrix A Columns, Connector_PinHeader_2.54mm:PinHeader_1x15_P2.54mm_Vertical, symbol Connector_Generic:Conn_01x15
- added J4: RGB LED Matrix A Rows, Connector_PinHeader_2.54mm:PinHeader_1x08_P2.54mm_Vertical, symbol Connector_Generic:Conn_01x08
- added J5: RGB LED Matrix B Columns, Connector_PinHeader_2.54mm:PinHeader_1x15_P2.54mm_Vertical, symbol Connector_Generic:Conn_01x15
- added J6: RGB LED Matrix B Rows, Connector_PinHeader_2.54mm:PinHeader_1x08_P2.54mm_Vertical, symbol Connector_Generic:Conn_01x08
- D1, D10, D11, D12, D13, D14, D15, D16, D17, D18, D19, D2, D20, D21, D22, D23, D24, D25, D26, D27, D28, D29, D3, D30, D31, D32, D33, D34, D35, D36, D37, D38, D39, D4, D40, D41, D42, D43, D44, D45, D46, D47, D48, D49, D5, D50, D51, D52, D53, D54, D55, D56, D57, D58, D59, D6, D60, D61, D62, D63, D64, D65, D66, D67, D68, D7, D8, D9: footprint Diode_SMD:D_0805_2012Metric -> Diode_SMD:D_1206_3216Metric
- D101, D102, D103, D104, D105, D106, D107, D108, D109, D110, D111, D112, D113, D114, D115, D116, D117, D118, D119, D120, D121, D122, D123, D124, D125, D126, D127, D128, D129, D130, D131, D132, D133, D134, D135, D136, D137, D138, D139, D140, D141, D142, D143, D144, D145, D146, D147, D148, D149, D150, D151, D152, D153, D154, D155, D156, D157, D158, D159, D160, D161, D162, D163, D164, D165, D166, D167, D168: footprint (none) -> dev-68:Wurth_PLCC6
Connections:
- net LED_A_COL_0: now also J3.1 (Pin_1); no longer U1.16 (CS1)
- net LED_A_COL_1: now also J3.2 (Pin_2); no longer U1.17 (CS2)
- net LED_A_COL_10: now also J3.11 (Pin_11); no longer U1.27 (CS11)
- net LED_A_COL_11: now also J3.12 (Pin_12); no longer U1.28 (CS12)
- net LED_A_COL_12: now also J3.13 (Pin_13); no longer U1.30 (CS13)
- net LED_A_COL_13: now also J3.14 (Pin_14); no longer U1.31 (CS14)
- net LED_A_COL_14: now also J3.15 (Pin_15); no longer U1.32 (CS15)
- net LED_A_COL_2: now also J3.3 (Pin_3); no longer U1.18 (CS3)
- net LED_A_COL_3: now also J3.4 (Pin_4); no longer U1.19 (CS4)
- net LED_A_COL_4: now also J3.5 (Pin_5); no longer U1.21 (CS5)
- net LED_A_COL_5: now also J3.6 (Pin_6); no longer U1.22 (CS6)
- net LED_A_COL_6: now also J3.7 (Pin_7); no longer U1.23 (CS7)
- net LED_A_COL_7: now also J3.8 (Pin_8); no longer U1.24 (CS8)
- net LED_A_COL_8: now also J3.9 (Pin_9); no longer U1.25 (CS9)
- net LED_A_COL_9: now also J3.10 (Pin_10); no longer U1.26 (CS10)
- net LED_A_ROW_0: now also J4.1 (Pin_1); no longer U1.2 (SW1)
- net LED_A_ROW_1: now also J4.2 (Pin_2); no longer U1.3 (SW2)
- net LED_A_ROW_2: now also J4.3 (Pin_3); no longer U1.4 (SW3)
- net LED_A_ROW_3: now also J4.4 (Pin_4); no longer U1.6 (SW4)
- net LED_A_ROW_4: now also J4.5 (Pin_5); no longer U1.7 (SW5)
- net LED_A_ROW_5: now also J4.6 (Pin_6); no longer U1.8 (SW6)
- net LED_A_ROW_6: now also J4.7 (Pin_7); no longer U1.9 (SW7)
- net LED_A_ROW_7: now also J4.8 (Pin_8); no longer U1.10 (SW8)
- net LED_B_COL_0: now also J5.1 (Pin_1); no longer U2.16 (CS1)
- net LED_B_COL_1: now also J5.2 (Pin_2); no longer U2.17 (CS2)
- net LED_B_COL_10: now also J5.11 (Pin_11); no longer U2.27 (CS11)
- net LED_B_COL_11: now also J5.12 (Pin_12); no longer U2.28 (CS12)
- net LED_B_COL_12: now also J5.13 (Pin_13); no longer U2.30 (CS13)
- net LED_B_COL_13: now also J5.14 (Pin_14); no longer U2.31 (CS14)
- net LED_B_COL_14: now also J5.15 (Pin_15); no longer U2.32 (CS15)
- net LED_B_COL_2: now also J5.3 (Pin_3); no longer U2.18 (CS3)
- net LED_B_COL_3: now also J5.4 (Pin_4); no longer U2.19 (CS4)
- net LED_B_COL_4: now also J5.5 (Pin_5); no longer U2.21 (CS5)
- net LED_B_COL_5: now also J5.6 (Pin_6); no longer U2.22 (CS6)
- net LED_B_COL_6: now also J5.7 (Pin_7); no longer U2.23 (CS7)
- net LED_B_COL_7: now also J5.8 (Pin_8); no longer U2.24 (CS8)
- net LED_B_COL_8: now also J5.9 (Pin_9); no longer U2.25 (CS9)
- net LED_B_COL_9: now also J5.10 (Pin_10); no longer U2.26 (CS10)
- net LED_B_ROW_0: now also J6.1 (Pin_1); no longer U2.2 (SW1)
- net LED_B_ROW_1: now also J6.2 (Pin_2); no longer U2.3 (SW2)
- net LED_B_ROW_2: now also J6.3 (Pin_3); no longer U2.4 (SW3)
- net LED_B_ROW_3: now also J6.4 (Pin_4); no longer U2.6 (SW4)
- net LED_B_ROW_4: now also J6.5 (Pin_5); no longer U2.7 (SW5)
- net LED_B_ROW_5: now also J6.6 (Pin_6); no longer U2.8 (SW6)
- net LED_B_ROW_6: now also J6.7 (Pin_7); no longer U2.9 (SW7)
- net LED_B_ROW_7: now also J6.8 (Pin_8); no longer U2.10 (SW8)
Other:
- moved on the sheet: U1, U2

Commit message: Better placement
Parts:
- removed J3: RGB LED Matrix A Columns, Connector_PinHeader_2.54mm:PinHeader_1x15_P2.54mm_Vertical, symbol Connector_Generic:Conn_01x15
- removed J4: RGB LED Matrix A Rows, Connector_PinHeader_2.54mm:PinHeader_1x08_P2.54mm_Vertical, symbol Connector_Generic:Conn_01x08
- added J3: RGB LED Matrix A Columns, Connector_PinHeader_2.54mm:PinHeader_2x16_P2.54mm_Vertical, symbol Connector_Generic:Conn_02x16_Odd_Even
- added J4: RGB LED Matrix A Rows, Connector_PinHeader_2.54mm:PinHeader_2x12_P2.54mm_Vertical, symbol Connector_Generic:Conn_02x12_Odd_Even
- added J7: LED Drivers, Connector_PinHeader_2.54mm:PinHeader_1x04_P2.54mm_Vertical, symbol Connector_Generic:Conn_01x04
- added J8: Power, Connector_PinHeader_2.54mm:PinHeader_1x04_P2.54mm_Vertical, symbol Connector_Generic:Conn_01x04
- J5: footprint Connector_PinHeader_2.54mm:PinHeader_1x15_P2.54mm_Vertical -> Connector_PinHeader_2.54mm:PinHeader_2x16_P2.54mm_Vertical; symbol Connector_Generic:Conn_01x15 -> Connector_Generic:Conn_02x16_Odd_Even
- J6: footprint Connector_PinHeader_2.54mm:PinHeader_1x08_P2.54mm_Vertical -> Connector_PinHeader_2.54mm:PinHeader_2x12_P2.54mm_Vertical; symbol Connector_Generic:Conn_01x08 -> Connector_Generic:Conn_02x12_Odd_Even
Connections:
- net LED_A_COL_0: now also J3.1 (Pin_1)
- net LED_A_COL_1: now also J3.3 (Pin_3)
- net LED_A_COL_10: now also J3.21 (Pin_21)
- net LED_A_COL_11: now also J3.23 (Pin_23)
- net LED_A_COL_12: now also J3.25 (Pin_25)
- net LED_A_COL_13: now also J3.27 (Pin_27)
- net LED_A_COL_14: now also J3.29 (Pin_29)
- net LED_A_COL_2: now also J3.5 (Pin_5)
- net LED_A_COL_3: now also J3.7 (Pin_7)
- net LED_A_COL_4: now also J3.9 (Pin_9)
- net LED_A_COL_5: now also J3.11 (Pin_11)
- net LED_A_COL_6: now also J3.13 (Pin_13)
- net LED_A_COL_7: now also J3.15 (Pin_15)
- net LED_A_COL_8: now also J3.17 (Pin_17)
- net LED_A_COL_9: now also J3.19 (Pin_19)
- net LED_A_ROW_0: now also J4.1 (Pin_1)
- net LED_A_ROW_1: now also J4.3 (Pin_3)
- net LED_A_ROW_2: now also J4.5 (Pin_5)
- net LED_A_ROW_3: now also J4.7 (Pin_7)
- net LED_A_ROW_4: now also J4.9 (Pin_9)
- net LED_A_ROW_5: now also J4.11 (Pin_11)
- net LED_A_ROW_6: now also J4.13 (Pin_13)
- net LED_A_ROW_7: now also J4.15 (Pin_15)
- net LED_B_COL_1: now also J5.3 (Pin_3); no longer J5.2 (Pin_2)
- net LED_B_COL_10: now also J5.21 (Pin_21); no longer J5.11 (Pin_11)
- net LED_B_COL_11: now also J5.23 (Pin_23); no longer J5.12 (Pin_12)
- net LED_B_COL_12: now also J5.25 (Pin_25); no longer J5.13 (Pin_13)
- net LED_B_COL_13: now also J5.27 (Pin_27); no longer J5.14 (Pin_14)
- net LED_B_COL_14: now also J5.29 (Pin_29); no longer J5.15 (Pin_15)
- net LED_B_COL_2: now also J5.5 (Pin_5); no longer J5.3 (Pin_3)
- net LED_B_COL_3: now also J5.7 (Pin_7); no longer J5.4 (Pin_4)
- net LED_B_COL_4: now also J5.9 (Pin_9); no longer J5.5 (Pin_5)
- net LED_B_COL_5: now also J5.11 (Pin_11); no longer J5.6 (Pin_6)
- net LED_B_COL_6: now also J5.13 (Pin_13); no longer J5.7 (Pin_7)
- net LED_B_COL_7: now also J5.15 (Pin_15); no longer J5.8 (Pin_8)
- net LED_B_COL_8: now also J5.17 (Pin_17); no longer J5.9 (Pin_9)
- net LED_B_COL_9: now also J5.19 (Pin_19); no longer J5.10 (Pin_10)
- net LED_B_ROW_1: now also J6.3 (Pin_3); no longer J6.2 (Pin_2)
- net LED_B_ROW_2: now also J6.5 (Pin_5); no longer J6.3 (Pin_3)
- net LED_B_ROW_3: now also J6.7 (Pin_7); no longer J6.4 (Pin_4)
- net LED_B_ROW_4: now also J6.9 (Pin_9); no longer J6.5 (Pin_5)
- net LED_B_ROW_5: now also J6.11 (Pin_11); no longer J6.6 (Pin_6)
- net LED_B_ROW_6: now also J6.13 (Pin_13); no longer J6.7 (Pin_7)
- net LED_B_ROW_7: now also J6.15 (Pin_15); no longer J6.8 (Pin_8)
- net A_SW8: now reaches U1.10 (SW8)
- net A_SW8: now also J4.16 (Pin_16)
- net A_SW9: now reaches U1.11 (SW9)
- net A_SW9: now also J4.18 (Pin_18)
- net A_SW10: now reaches U1.13 (SW10)
- net A_SW10: now also J4.20 (Pin_20)
- net A_SW11: now reaches U1.14 (SW11)
- net A_SW11: now also J4.22 (Pin_22)
- net A_SW12: now reaches U1.15 (SW12)
- net A_SW12: now also J4.24 (Pin_24)
- net A_CS1: now reaches U1.16 (CS1)
- net A_CS1: now also J3.2 (Pin_2)
- net A_CS2: now reaches U1.17 (CS2)
- net A_CS2: now also J3.4 (Pin_4)
- net A_CS3: now reaches U1.18 (CS3)
- net A_CS3: now also J3.6 (Pin_6)
- net A_CS4: now reaches U1.19 (CS4)
- net A_CS4: now also J3.8 (Pin_8)
- net A_SW1: now reaches U1.2 (SW1)
- net A_SW1: now also J4.2 (Pin_2)
- net A_CS5: now reaches U1.21 (CS5)
- net A_CS5: now also J3.10 (Pin_10)
- net A_CS6: now reaches U1.22 (CS6)
- net A_CS6: now also J3.12 (Pin_12)
- net A_CS7: now reaches U1.23 (CS7)
- net A_CS7: now also J3.14 (Pin_14)
- net A_CS8: now reaches U1.24 (CS8)
- net A_CS8: now also J3.16 (Pin_16)
- net A_CS9: now reaches U1.25 (CS9)
- net A_CS9: now also J3.18 (Pin_18)
- net A_CS10: now reaches U1.26 (CS10)
- net A_CS10: now also J3.20 (Pin_20)
- net A_CS11: now reaches U1.27 (CS11)
- net A_CS11: now also J3.22 (Pin_22)
- net A_CS12: now reaches U1.28 (CS12)
- net A_CS12: now also J3.24 (Pin_24)
- net A_SW2: now reaches U1.3 (SW2)
- net A_SW2: now also J4.4 (Pin_4)
- net A_CS13: now reaches U1.30 (CS13)
- net A_CS13: now also J3.26 (Pin_26)
- net A_CS14: now reaches U1.31 (CS14)
- net A_CS14: now also J3.28 (Pin_28)
- net A_CS15: now reaches U1.32 (CS15)
- net A_CS15: now also J3.30 (Pin_30)
- net A_CS16: now reaches U1.33 (CS16)
- net A_CS16: now also J3.32 (Pin_32)
- net A_SW3: now reaches U1.4 (SW3)
- net A_SW3: now also J4.6 (Pin_6)
- net SDA: now reaches U1.41 (SDA)
- net SDA: now also U2.41 (SDA), J7.1 (Pin_1)
- net SCL: now reaches U1.42 (SCL)
- net SCL: now also U2.42 (SCL), J7.2 (Pin_2)
- net INTB: now reaches U1.45 (~INTB)
- net INTB: now also U2.45 (~INTB), J7.3 (Pin_3)
- net SDB: now reaches U1.46 (~SDB)
- net SDB: now also U2.46 (~SDB), J7.4 (Pin_4)
- net A_SW4: now reaches U1.6 (SW4)
- net A_SW4: now also J4.8 (Pin_8)
- net A_SW5: now reaches U1.7 (SW5)
- net A_SW5: now also J4.10 (Pin_10)
- net A_SW6: now reaches U1.8 (SW6)
- net A_SW6: now also J4.12 (Pin_12)
- net A_SW7: now reaches U1.9 (SW7)
- net A_SW7: now also J4.14 (Pin_14)
- net B_SW8: now reaches U2.10 (SW8)
- net B_SW8: now also J6.16 (Pin_16)
- net B_SW9: now reaches U2.11 (SW9)
- net B_SW9: now also J6.18 (Pin_18)
- net B_SW10: now reaches U2.13 (SW10)
- net B_SW10: now also J6.20 (Pin_20)
- net B_SW11: now reaches U2.14 (SW11)
- net B_SW11: now also J6.22 (Pin_22)
- net B_SW12: now reaches U2.15 (SW12)
- net B_SW12: now also J6.24 (Pin_24)
- net B_CS1: now reaches U2.16 (CS1)
- net B_CS1: now also J5.2 (Pin_2)
- net B_CS2: now reaches U2.17 (CS2)
- net B_CS2: now also J5.4 (Pin_4)
- net B_CS3: now reaches U2.18 (CS3)
- net B_CS3: now also J5.6 (Pin_6)
- net B_CS4: now reaches U2.19 (CS4)
- net B_CS4: now also J5.8 (Pin_8)
- net B_SW1: now reaches U2.2 (SW1)
- net B_SW1: now also J6.2 (Pin_2)
- net B_CS5: now reaches U2.21 (CS5)
- net B_CS5: now also J5.10 (Pin_10)
- net B_CS6: now reaches U2.22 (CS6)
- net B_CS6: now also J5.12 (Pin_12)
- net B_CS7: now reaches U2.23 (CS7)
- net B_CS7: now also J5.14 (Pin_14)
- net B_CS8: now reaches U2.24 (CS8)
- net B_CS8: now also J5.16 (Pin_16)
- net B_CS9: now reaches U2.25 (CS9)
- net B_CS9: now also J5.18 (Pin_18)
- net B_CS10: now reaches U2.26 (CS10)
- net B_CS10: now also J5.20 (Pin_20)
- net B_CS11: now reaches U2.27 (CS11)
- net B_CS11: now also J5.22 (Pin_22)
- net B_CS12: now reaches U2.28 (CS12)
- net B_CS12: now also J5.24 (Pin_24)
- net B_SW2: now reaches U2.3 (SW2)
- net B_SW2: now also J6.4 (Pin_4)
- net B_CS13: now reaches U2.30 (CS13)
- net B_CS13: now also J5.26 (Pin_26)
- net B_CS14: now reaches U2.31 (CS14)
- net B_CS14: now also J5.28 (Pin_28)
- net B_CS15: now reaches U2.32 (CS15)
- net B_CS15: now also J5.30 (Pin_30)
- net B_CS16: now reaches U2.33 (CS16)
- net B_CS16: now also J5.32 (Pin_32)
- net B_SW3: now reaches U2.4 (SW3)
- net B_SW3: now also J6.6 (Pin_6)
- net B_SW4: now reaches U2.6 (SW4)
- net B_SW4: now also J6.8 (Pin_8)
- net B_SW5: now reaches U2.7 (SW5)
- net B_SW5: now also J6.10 (Pin_10)
- net B_SW6: now reaches U2.8 (SW6)
- net B_SW6: now also J6.12 (Pin_12)
- net B_SW7: now reaches U2.9 (SW7)
- net B_SW7: now also J6.14 (Pin_14)
- net COL0 renamed COL_0
- net COL1 renamed COL_1
- net COL2 renamed COL_2
- net COL3 renamed COL_3
- net COL4 renamed COL_4
- net COL5 renamed COL_5
- net COL6 renamed COL_6
- net COL7 renamed COL_7
- net ROW0 renamed ROW_0
- net ROW1 renamed ROW_1
- net ROW2 renamed ROW_2
- net ROW3 renamed ROW_3
- net ROW4 renamed ROW_4
- net ROW5 renamed ROW_5
- net ROW6 renamed ROW_6
- net ROW7 renamed ROW_7
- net ROW8 renamed ROW_8
- net ROW9 renamed ROW_9
- no-connect marks 0 -> 32
Other:
- moved on the sheet: U2

Commit message: Update schematic with all required 3733 components
Parts:
- added C1, C2: 22uF/10V, symbol Device:CP1_Small
- added C10, C11, C12, C13, C14, C9: 0.1uF, symbol Device:C_Small
- added C15, C16, C3, C4, C5, C6, C7, C8: 0.47uF, symbol Device:C_Small
- added R1, R4, R5: 100k, symbol Device:R_Small_US
- added R2, R3: 1k, symbol Device:R_Small_US
- added R6, R7: 20k, symbol Device:R_Small_US
- J7, J8: footprint Connector_PinHeader_2.54mm:PinHeader_1x04_P2.54mm_Vertical -> Connector_PinHeader_2.54mm:PinHeader_1x05_P2.54mm_Vertical; symbol Connector_Generic:Conn_01x04 -> Connector_Generic:Conn_01x05
Connections:
- net INTB: now also R1.2
- net SCL: now also J7.4 (Pin_4), R2.2; no longer J7.2 (Pin_2)
- net SDA: now also J7.5 (Pin_5), R3.2; no longer J7.1 (Pin_1)
- net SDB: now also J7.2 (Pin_2), R4.1; no longer J7.4 (Pin_4)
- net VCC: now reaches J8.1 (Pin_1)
- net VCC: now also J8.2 (Pin_2), U1.20 (PVCC), U1.29 (PVCC), U1.37 (AVCC), U1.38 (DVCC), U2.20 (PVCC), U2.29 (PVCC), U2.37 (AVCC), U2.38 (DVCC), U2.43 (ADDR1), C1.1, C10.2, C11.2, C12.2, C13.2, C14.2, C2.1, C3.2, C4.2, C5.2, C6.2, C7.2, C8.2, C9.2
- net GND: now reaches J8.3 (Pin_3)
- net GND: now also J8.4 (Pin_4), U1.12 (PGND), U1.34 (AGND), U1.43 (ADDR1), U1.44 (ADDR2), U1.48 (GND), U1.49 (GND), U1.5 (PGND), U2.12 (PGND), U2.34 (AGND), U2.44 (ADDR2), U2.48 (GND), U2.49 (GND), U2.5 (PGND), C1.2, C10.1, C11.1, C12.1, C13.1, C14.1, C15.2, C16.2, C2.2, C3.1, C4.1, C5.1, C6.1, C7.1, C8.1, C9.1, R4.2, R5.2, R6.2, R7.2
- net at U1.35 (RSET): now also R6.1
- net VIO: now reaches U1.39 (VIO)
- net VIO: now also J8.5 (Pin_5), U2.39 (VIO), C15.1, C16.1, R1.1, R2.1, R3.1
- net SYNC: now reaches U1.40 (SYNC)
- net SYNC: now also U2.40 (SYNC)
- net IICRST: now reaches U1.47 (IICRST)
- net IICRST: now also J7.1 (Pin_1), U2.47 (IICRST), R5.1
- net at U2.35 (RSET): now also R7.1
- no-connect marks 32 -> 10
Other:
- moved on the sheet: J3, J4, J5, J6, U1, U2

Commit message: Footprints for 3733 components
Parts:
- C1, C2: footprint (none) -> Capacitor_THT:CP_Radial_D4.0mm_P1.50mm
- C10, C11, C12, C13, C14, C15, C16, C3, C4, C5, C6, C7, C8, C9: footprint (none) -> Capacitor_SMD:C_1206_3216Metric_Pad1.42x1.75mm_HandSolder
- D1, D10, D11, D12, D13, D14, D15, D16, D17, D18, D19, D2, D20, D21, D22, D23, D24, D25, D26, D27, D28, D29, D3, D30, D31, D32, D33, D34, D35, D36, D37, D38, D39, D4, D40, D41, D42, D43, D44, D45, D46, D47, D48, D49, D5, D50, D51, D52, D53, D54, D55, D56, D57, D58, D59, D6, D60, D61, D62, D63, D64, D65, D66, D67, D68, D7, D8, D9: footprint Diode_SMD:D_1206_3216Metric -> Diode_SMD:D_1206_3216Metric_Pad1.42x1.75mm_HandSolder
- R1, R2, R3, R4, R5, R6, R7: footprint (none) -> Resistor_SMD:R_1206_3216Metric_Pad1.42x1.75mm_HandSolder

Commit message: some driver tracing
Connections:
- net IICRST: now also J7.5 (Pin_5); no longer J7.1 (Pin_1)
- net SCL: now also J7.2 (Pin_2); no longer J7.4 (Pin_4)
- net SDA: now also J7.1 (Pin_1); no longer J7.5 (Pin_5)
- net SDB: now also J7.4 (Pin_4); no longer J7.2 (Pin_2)
Changed lines of the file:
@@
 F 3 "~" H -7250 7500 50  0001 C CNN
 	1    -7250 7500
-	-1   0    0    1
+	-1   0    0    -1
 $EndComp
 Text GLabel -5800 7300 2    50   Input ~ 0
