File: dev-68.kicad_pcb (KiCad board)
At the start: 2 copper layers, 328.7 x 100.6 mm, 138 parts, among them J1 Columns, J2 Rows

Commit message: Some tracing
Parts:
- added D101: LED_RGB, dev-68:Wurth_PLCC6, F.Cu at (25.4, 19.8)
- added D102: LED_RGB, dev-68:Wurth_PLCC6, F.Cu at (44.5, 19.8)
- added D103: LED_RGB, dev-68:Wurth_PLCC6, F.Cu at (63.5, 19.8)
- added D104: LED_RGB, dev-68:Wurth_PLCC6, F.Cu at (82.5, 19.8)
- added D105: LED_RGB, dev-68:Wurth_PLCC6, F.Cu at (101.6, 19.8)
- added D106: LED_RGB, dev-68:Wurth_PLCC6, F.Cu at (120.7, 19.8)
- added D107: LED_RGB, dev-68:Wurth_PLCC6, F.Cu at (139.7, 19.8)
- added D108: LED_RGB, dev-68:Wurth_PLCC6, F.Cu at (158.8, 19.8)
- added D109: LED_RGB, dev-68:Wurth_PLCC6, F.Cu at (177.8, 19.8)
- added D110: LED_RGB, dev-68:Wurth_PLCC6, F.Cu at (196.8, 19.8)
- added D111: LED_RGB, dev-68:Wurth_PLCC6, F.Cu at (215.9, 19.8)
- added D112: LED_RGB, dev-68:Wurth_PLCC6, F.Cu at (234.9, 19.8)
- added D113: LED_RGB, dev-68:Wurth_PLCC6, F.Cu at (254.0, 19.8)
- added D114: LED_RGB, dev-68:Wurth_PLCC6, F.Cu at (282.6, 19.8)
- added D115: LED_RGB, dev-68:Wurth_PLCC6, F.Cu at (315.9, 19.8)
- added D116: LED_RGB, dev-68:Wurth_PLCC6, F.Cu at (335.0, 19.8)
- added D117: LED_RGB, dev-68:Wurth_PLCC6, F.Cu at (30.2, 38.9)
- added D118: LED_RGB, dev-68:Wurth_PLCC6, F.Cu at (54.0, 38.9)
- added D119: LED_RGB, dev-68:Wurth_PLCC6, F.Cu at (73.0, 38.9)
- added D120: LED_RGB, dev-68:Wurth_PLCC6, F.Cu at (92.1, 38.9)
- added D121: LED_RGB, dev-68:Wurth_PLCC6, F.Cu at (111.1, 38.9)
- added D122: LED_RGB, dev-68:Wurth_PLCC6, F.Cu at (130.2, 38.9)
- added D123: LED_RGB, dev-68:Wurth_PLCC6, F.Cu at (149.2, 38.9)
- added D124: LED_RGB, dev-68:Wurth_PLCC6, F.Cu at (168.3, 38.9)
- added D125: LED_RGB, dev-68:Wurth_PLCC6, F.Cu at (187.3, 38.9)
- added D126: LED_RGB, dev-68:Wurth_PLCC6, F.Cu at (206.4, 38.9)
- added D127: LED_RGB, dev-68:Wurth_PLCC6, F.Cu at (225.4, 38.9)
- added D128: LED_RGB, dev-68:Wurth_PLCC6, F.Cu at (244.5, 38.9)
- added D129: LED_RGB, dev-68:Wurth_PLCC6, F.Cu at (263.5, 38.9)
- added D130: LED_RGB, dev-68:Wurth_PLCC6, F.Cu at (287.3, 38.9)
- added D131: LED_RGB, dev-68:Wurth_PLCC6, F.Cu at (315.9, 38.9)
- added D132: LED_RGB, dev-68:Wurth_PLCC6, F.Cu at (335.0, 38.9)
- added D133: LED_RGB, dev-68:Wurth_PLCC6, F.Cu at (32.5, 57.9)
- added D134: LED_RGB, dev-68:Wurth_PLCC6, F.Cu at (58.7, 57.9)
- added D135: LED_RGB, dev-68:Wurth_PLCC6, F.Cu at (77.8, 57.9)
- added D136: LED_RGB, dev-68:Wurth_PLCC6, F.Cu at (96.8, 57.9)
- added D137: LED_RGB, dev-68:Wurth_PLCC6, F.Cu at (115.9, 57.9)
- added D138: LED_RGB, dev-68:Wurth_PLCC6, F.Cu at (134.9, 57.9)
- added D139: LED_RGB, dev-68:Wurth_PLCC6, F.Cu at (154.0, 57.9)
- added D140: LED_RGB, dev-68:Wurth_PLCC6, F.Cu at (173.0, 57.9)
- added D141: LED_RGB, dev-68:Wurth_PLCC6, F.Cu at (192.1, 57.9)
- added D142: LED_RGB, dev-68:Wurth_PLCC6, F.Cu at (211.1, 57.9)
- added D143: LED_RGB, dev-68:Wurth_PLCC6, F.Cu at (230.2, 57.9)
- added D144: LED_RGB, dev-68:Wurth_PLCC6, F.Cu at (249.2, 57.9)
- added D145: LED_RGB, dev-68:Wurth_PLCC6, F.Cu at (280.2, 57.9)
- added D146: LED_RGB, dev-68:Wurth_PLCC6, F.Cu at (37.3, 77.0)
- added D147: LED_RGB, dev-68:Wurth_PLCC6, F.Cu at (68.3, 77.0)
- added D148: LED_RGB, dev-68:Wurth_PLCC6, F.Cu at (87.3, 77.0)
- added D149: LED_RGB, dev-68:Wurth_PLCC6, F.Cu at (106.4, 77.0)
- added D150: LED_RGB, dev-68:Wurth_PLCC6, F.Cu at (125.4, 77.0)
- added D151: LED_RGB, dev-68:Wurth_PLCC6, F.Cu at (144.5, 77.0)
- added D152: LED_RGB, dev-68:Wurth_PLCC6, F.Cu at (163.5, 77.0)
- added D153: LED_RGB, dev-68:Wurth_PLCC6, F.Cu at (182.6, 77.0)
- added D154: LED_RGB, dev-68:Wurth_PLCC6, F.Cu at (201.6, 77.0)
- added D155: LED_RGB, dev-68:Wurth_PLCC6, F.Cu at (220.7, 77.0)
- added D156: LED_RGB, dev-68:Wurth_PLCC6, F.Cu at (239.7, 77.0)
- added D157: LED_RGB, dev-68:Wurth_PLCC6, F.Cu at (275.4, 77.0)
- added D158: LED_RGB, dev-68:Wurth_PLCC6, F.Cu at (315.9, 77.0)
- added D159: LED_RGB, dev-68:Wurth_PLCC6, F.Cu at (27.8, 96.0)
- added D160: LED_RGB, dev-68:Wurth_PLCC6, F.Cu at (51.6, 96.0)
- added D161: LED_RGB, dev-68:Wurth_PLCC6, F.Cu at (75.4, 96.0)
- added D162: LED_RGB, dev-68:Wurth_PLCC6, F.Cu at (146.8, 96.0)
- added D163: LED_RGB, dev-68:Wurth_PLCC6, F.Cu at (218.3, 96.0)
- added D164: LED_RGB, dev-68:Wurth_PLCC6, F.Cu at (242.1, 96.0)
- added D165: LED_RGB, dev-68:Wurth_PLCC6, F.Cu at (265.9, 96.0)
- added D166: LED_RGB, dev-68:Wurth_PLCC6, F.Cu at (296.9, 96.0)
- added D167: LED_RGB, dev-68:Wurth_PLCC6, F.Cu at (315.9, 96.0)
- added D168: LED_RGB, dev-68:Wurth_PLCC6, F.Cu at (335.0, 96.0)
- added J3: RGB LED Matrix A Columns, Connector_PinHeader_2.54mm:PinHeader_1x15_P2.54mm_Vertical, F.Cu at (2.38, -6.35)
- added J4: RGB LED Matrix A Rows, Connector_PinHeader_2.54mm:PinHeader_1x08_P2.54mm_Vertical, F.Cu at (90.5, -14.3)
- added J5: RGB LED Matrix B Columns, Connector_PinHeader_2.54mm:PinHeader_1x15_P2.54mm_Vertical, F.Cu at (335.8, -23.0)
- added J6: RGB LED Matrix B Rows, Connector_PinHeader_2.54mm:PinHeader_1x08_P2.54mm_Vertical, F.Cu at (240.5, -26.2)
- added U1: IS31FL3733-TQ, Package_QFP:TQFP-48-1EP_7x7mm_P0.5mm_EP5x5mm, F.Cu at (50.8, -20.6)
- added U2: IS31FL3733-TQ, Package_QFP:TQFP-48-1EP_7x7mm_P0.5mm_EP5x5mm, F.Cu at (300.8, -30.2)
- D1, D10, D11, D12, D13, D14, D15, D16, D17, D18, D19, D2, D20, D21, D22, D23, D24, D25, D26, D27, D28, D29, D3, D30, D31, D32, D33, D34, D35, D36, D37, D38, D39, D4, D40, D41, D42, D43, D44, D45, D46, D47, D48, D49, D5, D50, D51, D52, D53, D54, D55, D56, D57, D58, D59, D6, D60, D61, D62, D63, D64, D65, D66, D67, D68, D7, D8, D9: footprint Diode_SMD:D_0805_2012Metric -> Diode_SMD:D_1206_3216Metric; moved to F.Cu
- moved J1 36.3 mm to (163.5, -21.4)
- moved J2 36.3 mm to (184.2, -21.4)
- moved D59 16.1 mm to (22.2, 109.5), turned to 180 degrees
- moved D41 5.78 mm to (182.6, 70.6), turned to 90 degrees
- moved D54 5.78 mm to (192.1, 89.7), turned to 90 degrees
- moved D9 5.78 mm to (168.3, 32.5), turned to 90 degrees
- moved D25 5.78 mm to (177.8, 51.6), turned to 90 degrees
- moved D60 2.25 mm to (39.7, 108.7)
- moved D33 1.83 mm to (27.0, 71.4)
- moved D17 1.77 mm to (24.6, 52.4)
- moved D67 1.77 mm to (306.4, 108.7)
- moved D68 1.77 mm to (325.4, 108.7)
- moved D1 1.77 mm to (19.8, 33.3)
- moved D46 1.77 mm to (31.8, 90.5)
- moved D64 1.73 mm to (230.2, 108.9)
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Routing:
- net COL0: track 485.8 -> 161.3 mm, vias 13 -> 0
- net COL1: track 456.8 -> 169.2 mm, vias 15 -> 0
- net COL2: track 422.4 -> 185.7 mm, vias 17 -> 0
- net ROW8: track 373.8 -> 147.7 mm
- net ROW5: track 311.9 -> 119.1 mm
- net COL3: track 278.3 -> 90.0 mm, vias 9 -> 0
- net ROW1: track 302.4 -> 132.9 mm
- net ROW0: track 297.6 -> 128.2 mm
- net ROW2: track 304.7 -> 135.4 mm
- net ROW3: track 311.0 -> 141.8 mm
- net COL4: track 308.9 -> 157.2 mm, vias 13 -> 0
- net COL5: track 289.1 -> 174.1 mm, vias 17 -> 0
- net LED_B_ROW_5: track 0.00 -> 105.8 mm, vias 0 -> 8
- net LED_A_ROW_1: track 0.00 -> 98.6 mm, vias 0 -> 8
- net LED_A_ROW_2: track 0.00 -> 96.7 mm, vias 0 -> 8
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Other:
- board outline removed

Commit message: Undo some traces; do just the "easy" traces.
Routing:
- net LED_B_ROW_5: track 105.8 -> 8.50 mm, vias 8 -> 0
- net LED_A_ROW_1: track 98.6 -> 8.50 mm, vias 8 -> 0
- net LED_A_ROW_2: track 96.7 -> 8.50 mm, vias 8 -> 0
- net LED_B_ROW_3: track 94.5 -> 6.80 mm, vias 6 -> 0
- net LED_B_ROW_1: track 92.7 -> 8.50 mm, vias 8 -> 0
- net LED_B_ROW_2: track 92.3 -> 8.50 mm, vias 8 -> 0
- net LED_A_ROW_5: track 92.1 -> 8.50 mm, vias 8 -> 0
- net LED_A_ROW_0: track 90.0 -> 8.50 mm, vias 8 -> 0
- net LED_B_ROW_7: track 80.7 -> 5.10 mm, vias 4 -> 0
- net LED_B_ROW_6: track 81.9 -> 6.80 mm, vias 6 -> 0
- net LED_B_ROW_0: track 71.6 -> 6.80 mm, vias 6 -> 0
- net LED_A_ROW_3: track 71.4 -> 6.80 mm, vias 6 -> 0
- net LED_A_ROW_7: track 71.4 -> 6.80 mm, vias 6 -> 0
- net LED_A_ROW_4: track 71.4 -> 6.80 mm, vias 6 -> 0
- net LED_A_ROW_6: track 71.1 -> 6.80 mm, vias 6 -> 0
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
Commit message: Minimized vias
Parts:
- moved D25 0.16 mm to (177.8, 51.4)
- moved D64 0.14 mm to (230.2, 108.7)
Routing:
- net LED_B_ROW_5: track 8.50 -> 113.9 mm, vias 0 -> 5
- net LED_A_ROW_1: track 8.50 -> 108.0 mm, vias 0 -> 5
- net LED_A_ROW_2: track 8.50 -> 106.1 mm, vias 0 -> 5
- net LED_B_ROW_1: track 8.50 -> 103.9 mm, vias 0 -> 5
- net LED_B_ROW_3: track 6.80 -> 101.2 mm, vias 0 -> 4
- net LED_B_ROW_2: track 8.50 -> 102.1 mm, vias 0 -> 5
- net LED_A_ROW_5: track 8.50 -> 102.1 mm, vias 0 -> 5
- net LED_A_ROW_0: track 8.50 -> 100.2 mm, vias 0 -> 5
- net LED_B_ROW_6: track 6.80 -> 93.4 mm, vias 0 -> 4
- net LED_B_ROW_7: track 5.10 -> 88.7 mm, vias 0 -> 3
- net LED_A_ROW_6: track 6.80 -> 79.1 mm, vias 0 -> 4
- net LED_A_ROW_3: track 6.80 -> 79.1 mm, vias 0 -> 4
- net LED_B_ROW_0: track 6.80 -> 79.1 mm, vias 0 -> 4
- net LED_A_ROW_7: track 6.80 -> 79.1 mm, vias 0 -> 4
- net LED_A_ROW_4: track 6.80 -> 79.1 mm, vias 0 -> 4
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
Commit message: RGB LED traces
Parts:
- moved J1 167.5 mm to (161.0, 146.0)
- moved J2 167.5 mm to (181.7, 146.0)
- moved J4 167.5 mm to (88.0, 153.2)
- moved J6 167.5 mm to (238.0, 141.3)
- moved J5 73.4 mm to (364.5, 44.6), turned to 0 degrees
- moved J3 50.5 mm to (1.52, 44.1), turned to 0 degrees
Routing:
- net LED_B_COL_1: track 0.00 -> 165.6 mm
- net LED_B_COL_2: track 0.00 -> 164.2 mm
- net LED_B_COL_0: track 0.00 -> 163.7 mm
- net LED_B_COL_4: track 0.00 -> 156.0 mm
- net LED_B_COL_5: track 0.00 -> 155.3 mm
- net LED_A_COL_10: track 0.00 -> 153.7 mm
- net LED_A_COL_11: track 0.00 -> 152.9 mm
- net LED_B_COL_3: track 0.00 -> 151.1 mm
- net LED_A_COL_9: track 0.00 -> 150.2 mm
- net LED_A_COL_7: track 0.00 -> 148.9 mm
- net LED_A_COL_8: track 0.00 -> 147.8 mm
- net LED_A_COL_4: track 0.00 -> 146.5 mm
- net LED_A_COL_5: track 0.00 -> 144.5 mm
- net LED_A_COL_6: track 0.00 -> 144.0 mm
- net LED_A_COL_1: track 0.00 -> 141.8 mm
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
Commit message: so. many. traces...
Parts:
- moved J4 180.0 mm to (5.00, -6.50)
- moved J6 156.8 mm to (314.8, 4.50)
- moved J2 146.1 mm to (191.2, 0.25)
- moved J1 143.6 mm to (148.2, 3.00), turned to 90 degrees
Routing:
- net COL0: track 161.3 -> 609.2 mm, vias 0 -> 4
- net COL1: track 169.2 -> 543.4 mm, vias 0 -> 4
- net COL2: track 185.7 -> 492.1 mm, vias 0 -> 4
- net COL3: track 90.0 -> 363.9 mm, vias 0 -> 4
- net COL4: track 157.2 -> 365.1 mm, vias 0 -> 4
- net COL5: track 174.1 -> 327.9 mm, vias 0 -> 4
- net ROW4: track 115.3 -> 256.7 mm, vias 0 -> 1
- net ROW5: track 119.1 -> 236.6 mm, vias 0 -> 1
- net COL6: track 154.1 -> 253.2 mm, vias 0 -> 4
- net ROW3: track 141.8 -> 235.4 mm, vias 0 -> 1
- net ROW6: track 116.0 -> 202.8 mm, vias 0 -> 1
- net ROW2: track 135.4 -> 199.5 mm, vias 0 -> 1
- net ROW7: track 76.2 -> 140.0 mm, vias 0 -> 1
- net COL7: track 134.0 -> 183.5 mm, vias 0 -> 2
- net ROW1: track 132.9 -> 175.6 mm, vias 0 -> 1
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
Commit message: LED A Matrix + Rows and Cols
Parts:
- moved J3 70.1 mm to (53.2, -3.25), turned to 270 degrees
- moved J4 56.8 mm to (61.8, -3.25)
- moved J5 52.5 mm to (342.8, -3.25), turned to 270 degrees
- moved J1 44.4 mm to (104.2, -3.25)
- moved J2 39.7 mm to (151.8, -3.25)
- moved J6 34.9 mm to (280.8, -3.25)
- moved U2 8.09 mm to (302.5, -22.2)
- moved U1 7.04 mm to (57.8, -19.5)
Routing:
- net LED_A_ROW_7: track 79.1 -> 252.3 mm, vias 4 -> 6
- net LED_A_ROW_6: track 79.1 -> 232.7 mm, vias 4 -> 6
- net LED_A_ROW_5: track 102.1 -> 236.1 mm, vias 5 -> 7
- net LED_A_COL_14: track 122.0 -> 239.0 mm, vias 0 -> 1
- net LED_A_COL_13: track 122.7 -> 238.0 mm, vias 0 -> 1
- net LED_A_ROW_4: track 79.1 -> 193.3 mm, vias 4 -> 6
- net LED_A_COL_12: track 122.1 -> 235.2 mm, vias 0 -> 1
- net LED_A_COL_10: track 153.7 -> 255.8 mm, vias 0 -> 1
- net LED_A_COL_11: track 152.9 -> 255.1 mm, vias 0 -> 1
- net LED_A_COL_9: track 150.2 -> 251.8 mm, vias 0 -> 1
- net ROW0: track 148.1 -> 245.1 mm, vias 1 -> 3
- net LED_A_ROW_3: track 79.1 -> 173.5 mm, vias 4 -> 6
- net ROW9: track 178.6 -> 265.5 mm, vias 1 -> 3
- net LED_A_COL_8: track 147.8 -> 231.0 mm, vias 0 -> 1
- net LED_A_COL_7: track 148.9 -> 231.8 mm, vias 0 -> 1
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Other:
- board outline added: 340 x 147 mm

Commit message: Finished traces
Parts:
- moved J5 35.5 mm to (307.2, -3.25), turned to 90 degrees
Routing:
- net LED_B_COL_8: track 92.8 -> 228.2 mm, vias 0 -> 1
- net LED_B_COL_7: track 92.9 -> 227.6 mm, vias 0 -> 1
- net LED_B_COL_6: track 91.6 -> 225.9 mm, vias 0 -> 1
- net LED_B_ROW_0: track 79.1 -> 197.1 mm
- net LED_B_COL_11: track 119.0 -> 232.9 mm, vias 0 -> 1
- net LED_B_COL_10: track 119.1 -> 232.8 mm, vias 0 -> 1
- net LED_B_COL_9: track 119.3 -> 232.4 mm, vias 0 -> 1
- net LED_B_COL_14: track 122.0 -> 233.9 mm, vias 0 -> 1
- net LED_B_COL_13: track 122.7 -> 234.3 mm, vias 0 -> 1
- net LED_B_COL_12: track 119.2 -> 230.2 mm, vias 0 -> 1
- net LED_B_ROW_1: track 103.9 -> 207.2 mm
- net LED_B_ROW_2: track 102.1 -> 189.0 mm
- net LED_B_ROW_3: track 101.2 -> 166.8 mm
- net LED_B_COL_3: track 151.1 -> 213.3 mm, vias 0 -> 1
- net LED_B_COL_4: track 156.0 -> 217.8 mm, vias 0 -> 1
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